File: PCB/Popn2/pop_pico2.kicad_sch (KiCad schematic)
At the start: 55 parts, among them SW1 SW_DIP_x01, SW10 SW_DIP_x01, SW11 SW_DIP_x01, SW2 SW_DIP_x01, SW3 SW_DIP_x01, SW4 SW_DIP_x01, SW5 SW_DIP_x01, SW6 SW_DIP_x01, SW7 SW_DIP_x01, SW8 SW_DIP_x01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

Commit message: PCB v1.0
Parts:
- added C5, C6: 0.1uF, Capacitor_SMD:C_0603_1608Metric_Pad1.08x0.95mm_HandSolder, symbol Device:C
- SW1, SW2, SW3, SW4, SW5, SW6, SW7, SW8, SW9: footprint popn_pico2:SW_Kailh_Choc_V1V2_1.00u_LED -> popn_pico2:SW_Choc_V1V2_Cherry_MX_LED
- SW10, SW11: footprint Button_Switch_THT:SW_SPST_Omron_B3F-315x_Angled -> popn_pico2:Omron_B3F-315x_Angled
Connections:
- net +5V: now also C5.1, C6.1
- net GND: now also C5.2, C6.2
- net K10: now also U1.7 (GPIO5); no longer U1.31 (GPIO26_ADC0)
- net K11: now also U1.9 (GPIO6); no longer U1.32 (GPIO27_ADC1)
- net K2: now also U1.2 (GPIO1); no longer U1.4 (GPIO2)
- net K3: now also U1.4 (GPIO2); no longer U1.6 (GPIO4)
- net K4: now also U1.5 (GPIO3); no longer U1.9 (GPIO6)
- net K5: now also U1.6 (GPIO4); no longer U1.11 (GPIO8)
- net K6: now also U1.10 (GPIO7); no longer U1.14 (GPIO10)
- net K7: now also U1.11 (GPIO8); no longer U1.16 (GPIO12)
- net K8: now also U1.12 (GPIO9); no longer U1.19 (GPIO14)
- net K9: now also U1.14 (GPIO10); no longer U1.21 (GPIO16)
- net RGB2: now also U1.32 (GPIO27_ADC1); no longer U1.29 (GPIO22)
