File: PCB/Popn2/pop_pico2.kicad_pcb (KiCad board)
At the start: 2 copper layers, 297 x 114 mm, 55 parts, among them SW1 SW_DIP_x01, SW10 SW_DIP_x01, SW11 SW_DIP_x01, SW2 SW_DIP_x01, SW3 SW_DIP_x01, SW4 SW_DIP_x01, SW5 SW_DIP_x01, SW6 SW_DIP_x01, SW7 SW_DIP_x01, SW8 SW_DIP_x01, SW9 SW_DIP_x01, U1 PiPico_No_SWD

Commit message: PCB v1.0
Parts:
- added C5: 0.1uF, Capacitor_SMD:C_0603_1608Metric_Pad1.08x0.95mm_HandSolder, B.Cu at (275.4, 126.1)
- added C6: 0.1uF, Capacitor_SMD:C_0603_1608Metric_Pad1.08x0.95mm_HandSolder, B.Cu at (332.1, 122.0)
- C1, C2, C3, C4: moved to B.Cu
- SW1, SW2, SW3, SW4, SW5, SW6, SW7, SW8, SW9: footprint popn_pico2:SW_Kailh_Choc_V1V2_1.00u_LED -> popn_pico2:SW_Choc_V1V2_Cherry_MX_LED
- SW10, SW11: footprint Button_Switch_THT:SW_SPST_Omron_B3F-315x_Angled -> popn_pico2:Omron_B3F-315x_Angled
- moved D36 121.1 mm to (106.3, 105.3), turned to 60 degrees
- moved C3 94.3 mm to (216.2, 126.1)
- moved C4 71.7 mm to (284.5, 92.2)
- moved D35 68.4 mm to (162.3, 77.3), turned to 0 degrees
- moved D34 59.8 mm to (221.3, 77.3)
- moved C2 59.8 mm to (165.8, 92.2)
- moved C1 30.0 mm to (105.0, 121.1)
- moved D32 14.1 mm to (336.3, 105.3), turned to -60 degrees
- moved D28 10.0 mm to (132.8, 140.3)
- moved D29 10.0 mm to (191.8, 140.3)
- moved D30 10.0 mm to (250.8, 140.3)
- moved D31 10.0 mm to (309.8, 140.3)
- moved D33 10.0 mm to (280.3, 77.3)
- moved SW10 8.85 mm to (245.8, 54.3)
- moved SW11 5.28 mm to (264.3, 54.3)
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- renumbered D3 to D1, D21 to D10, D19 to D11, D20 to D12, D27 to D13, D25 to D14, D26 to D15, D23 to D16, D24 to D17, D22 to D18, D17 to D19, D1 to D2, D18 to D20, D16 to D21, D11 to D22, D12 to D23, D10 to D24, D5 to D25, D6 to D26, D4 to D27, D2 to D3, D9 to D4, D7 to D5, D8 to D6, D15 to D7, D13 to D8, D14 to D9
Connections:
- D1 pad I: Net-(D2-Out) (its old number) -> /RGB1
- D1 pad O: Net-(D3-Out) -> Net-(D1-Out)
- D10 pad I: Net-(D20-Out) -> Net-(D10-In)
- D10 pad O: Net-(D21-Out) -> Net-(D10-Out)
- D11 pad I: Net-(D18-Out) -> Net-(D10-Out)
- D12 pad O: Net-(D20-Out) -> Net-(D12-Out)
- D13 pad I: Net-(D26-Out) -> Net-(D12-Out)
- D13 pad O: unconnected-(D27-Out-PadO) -> Net-(D13-Out)
- D14 pad I: Net-(D24-Out) -> Net-(D13-Out)
- D15 pad O: Net-(D26-Out) -> Net-(D15-Out)
- D16 pad I: Net-(D22-Out) (its old number) -> Net-(D15-Out)
- D17 pad O: Net-(D24-Out) -> Net-(D17-Out)
- D18 pad I: Net-(D21-Out) -> Net-(D17-Out)
- D18 pad O: Net-(D22-Out) (its old number) -> Net-(D18-Out)
- D19 pad I: Net-(D16-Out) (its old number) -> Net-(D18-Out)
- D2 pad I: /RGB1 -> Net-(D1-Out)
- D20 pad O: Net-(D18-Out) -> Net-(D20-Out)
- D21 pad I: Net-(D15-Out) -> Net-(D20-Out)
- D21 pad O: Net-(D16-Out) (its old number) -> Net-(D21-Out)
- D22 pad I: Net-(D10-Out) -> Net-(D21-Out)
- D23 pad O: Net-(D12-Out) -> Net-(D23-Out)
- D24 pad I: Net-(D10-In) -> Net-(D23-Out)
- D24 pad O: Net-(D10-Out) -> Net-(D24-Out)
- D25 pad I: Net-(D4-Out) -> Net-(D24-Out)
- D26 pad O: Net-(D6-Out) -> Net-(D26-Out)
- D27 pad I: Net-(D3-Out) -> Net-(D26-Out)
- D27 pad O: Net-(D4-Out) -> unconnected-(D27-Out-PadO)
- D3 pad O: Net-(D2-Out) (its old number) -> Net-(D3-Out)
- D4 pad I: Net-(D8-Out) (its old number) -> Net-(D3-Out)
- D4 pad O: Net-(D10-In) -> Net-(D4-Out)
- D5 pad I: Net-(D6-Out) -> Net-(D4-Out)
- D6 pad O: Net-(D8-Out) (its old number) -> Net-(D6-Out)
- D7 pad I: Net-(D14-Out) (its old number) -> Net-(D6-Out)
- D7 pad O: Net-(D15-Out) -> Net-(D7-Out)
- D8 pad I: Net-(D12-Out) -> Net-(D7-Out)
- D9 pad O: Net-(D14-Out) (its old number) -> Net-(D10-In)
- U1 pad 10: unconnected-(U1-GPIO7-Pad10) -> /K6
- U1 pad 11: /K5 -> /K7
- U1 pad 12: unconnected-(U1-GPIO9-Pad12) -> /K8
- U1 pad 14: /K6 -> /K9
- U1 pad 16: /K7 -> unconnected-(U1-GPIO12-Pad16)
- U1 pad 19: /K8 -> unconnected-(U1-GPIO14-Pad19)
- U1 pad 2: unconnected-(U1-GPIO1-Pad2) -> /K2
- U1 pad 21: /K9 -> unconnected-(U1-GPIO16-Pad21)
- U1 pad 29: /RGB2 -> unconnected-(U1-GPIO22-Pad29)
- U1 pad 31: /K10 -> unconnected-(U1-GPIO26_ADC0-Pad31)
- U1 pad 32: /K11 -> /RGB2
- U1 pad 4: /K2 -> /K3
- U1 pad 5: unconnected-(U1-GPIO3-Pad5) -> /K4
- U1 pad 6: /K3 -> /K5
- U1 pad 7: unconnected-(U1-GPIO5-Pad7) -> /K10
- U1 pad 9: /K4 -> /K11
Routing:
- net +5V: track 0.00 -> 1054.2 mm, vias 0 -> 8
- net /K9: track 0.00 -> 140.5 mm, vias 0 -> 1
- net /RGB1: track 0.00 -> 114.3 mm, vias 0 -> 1
- net /K1: track 0.00 -> 110.9 mm, vias 0 -> 2
- net /K8: track 0.00 -> 103.7 mm, vias 0 -> 1
- net /RGB2: track 0.00 -> 101.9 mm, vias 0 -> 3
- net Net-(D31-Out): track 0.00 -> 91.0 mm
- net /K7: track 0.00 -> 88.6 mm, vias 0 -> 1
- net /K2: track 0.00 -> 87.5 mm, vias 0 -> 1
- net VBUS: track 0.00 -> 83.9 mm, vias 0 -> 2
- net Net-(D32-Out): track 0.00 -> 83.2 mm
- net Net-(D35-Out): track 0.00 -> 83.0 mm
- net /K11: track 0.00 -> 74.2 mm, vias 0 -> 1
- net /K3: track 0.00 -> 72.7 mm, vias 0 -> 1
- net /USB_DN: track 0.00 -> 70.5 mm
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- added copper zone on B.Cu, net GND
- added copper zone on F.Cu, net GND
Other:
- board size 297 x 114 mm -> 297 x 95 mm
- board text added: "Popn Pico 2"
- board text added: "v1.0"

Commit message: Optimize switch footprints
Other:
- board text added: "v1.1"
- board text removed: "v1.0"
